File: wwgt2026badge/wwgt2026badge.kicad_pcb (KiCad board)
At the start: 2 copper layers, 100 x 70 mm, 20 parts, among them J1 Conn_01x08_Pin, J2 Conn_01x04_Pin, SW1 SW_PUSH, SW2 EC12PLGRSDVF, SW3 SW_PUSH, U2 rp2040-zero, U3 fj08k-s

Commit message: added gbr files
Parts:
- moved REF** 1.25 mm to (80.5, 88.2)
